File: kicad/SamDrum/SamDrum.kicad_sch (KiCad schematic)
At the start: 11 parts

Commit message: Updated schematics
Parts:
- removed U?: LM324, symbol Amplifier_Operational:LM324
- added C? (x2): 1u, KOMA Parts:WIMA_1uF, symbol KomaFieldKit-PR3-rescue:C
- added D? (x2): D_Schottky, symbol Device:D_Schottky
- added J? (x2): AudioJack2, symbol Connector:AudioJack2
- added R? (x2): 1M, otto:SMD_0603, symbol KomaFieldKit-PR3-rescue:R
- added R? (x2): 100K, otto:SMD_0603, symbol KomaFieldKit-PR3-rescue:R
- added TP? (x2): 1V65, symbol Connector:TestPoint
- added TP?: To Bela Analog In 1 (pd: adc~ 4), symbol Connector:TestPoint
- added TP?: To Bela Analog In 2 (pd: adc~ 5), symbol Connector:TestPoint
- added U? (x3): LM324, otto:SOIC-14, symbol KomaFieldKit-PR3-rescue:LM324
- TP?: value To Bela ADC0 -> To Bela Analog In 0 (pd: adc~ 3)
Connections:
- net +3V3: now also D?.1 (K), D?.1 (K)
- net GND: now also J?.S, J?.S
- net at C?.2, R?.1: now also U?.3 (+)
- net at D?.2 (A), TP?.1: now also U?.1, U?.2 (-)
- new net: C?.2, J?.T, R?.2 (x2)
- new net: R?.1, TP?.1 (x2)
- new net: C?.1, R?.2, U?.3 (+) (x2)
- new net: D?.2 (A), TP?.1, U?.1, U?.2 (-) (x2)
- new net AGND: R?.1, R?.1
Other:
- note added: "Audio Audio Inputs"
- note added: "gain"
- note removed: "Audio Inputs"
- moved on the sheet: C?, D?, J?, R?, TP?
